File: PCB/HackPad1.kicad_pcb (KiCad board)
At the start: 2 copper layers, 69.8 x 60.5 mm, 19 parts, among them J1 Conn_01x04_Pin, SW1 SW_Push, SW10 RotaryEncoder, SW2 SW_Push, SW4 SW_Push, SW5 SW_Push, SW7 SW_Push, SW8 SW_Push, U1 MOUDLE-SEEEDUINO-XIAO

Commit message: COmpleted
Other:
- board size 69.8 x 60.5 mm -> 77.2 x 60.9 mm
Changed lines of the file:
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@@
 	)
 	(gr_rect
-		(start 97.25 46.25)
-		(end 167 106.75)
+		(start 97.25 45.875)
+		(end 174.45 106.75)
 		(stroke
 			(width 0.05)
